File: projects/Cat toy 1/wiring/wiring.kicad_sch (KiCad schematic)
At the start: 6 parts, among them M1 Stepper_Motor_bipolar, SW1 Limit switch (left), SW2 Limit switch (right)

Commit message: BeltDriver
Parts:
- removed C1: 100mF, symbol Device:C_Polarized
- removed SW1: Limit switch (left), symbol Switch:SW_SPDT
- removed SW2: Limit switch (right), symbol Switch:SW_SPDT
Connections:
- net +12V renamed +9V
- net Internal pullup resistor: no longer names the net of A3.7 (D4)
- net Internal pullup resistor: no longer A3.8 (D5)
