File: projects/StepperMotorArduino/wiring/wiring.kicad_pcb (KiCad board)
At the start: 2 copper layers, 136.9 x 42.3 mm, 12 parts, among them J1 Conn_01x02_Pin, J2 Conn_01x02_Pin, J3 Conn_01x02_Pin, J4 Conn_01x02_Pin, J5 Conn_01x04_Pin, J6 Conn_01x04_Pin, J7 Conn_01x02_Pin, U1 NRF24L01_Breakout

Commit message: Progress
Parts:
- removed the U1 at (149.1, 71.1)
- added C2: 0.1mF, Capacitor_THT:C_Radial_D6.3mm_H7.0mm_P2.50mm, F.Cu at (224.0, 90.5)
- added C3: 10mF, Capacitor_THT:CP_Radial_D8.0mm_P3.80mm, F.Cu at (182.1, 92.9)
- added C4: 0.1mF, Capacitor_THT:C_Radial_D6.3mm_H7.0mm_P2.50mm, F.Cu at (170.8, 92.5)
- added C5: 100mF, Capacitor_THT:CP_Radial_D8.0mm_P3.80mm, F.Cu at (196.0, 61.3)
- added C6: 0.1mF, Capacitor_THT:C_Radial_D6.3mm_H7.0mm_P2.50mm, F.Cu at (166.4, 60.2)
- added C8: 100mF, Capacitor_THT:CP_Radial_D8.0mm_P3.80mm, F.Cu at (157.8, 61.2)
- added J8: Conn_01x02_Pin, Connector_PinSocket_2.54mm:PinSocket_1x02_P2.54mm_Vertical, F.Cu at (200.4, 73.7)
- added J9: Conn_01x02_Pin, Connector_PinSocket_2.54mm:PinSocket_1x02_P2.54mm_Vertical, F.Cu at (177.3, 79.5)
- added U2: Mini560-pro-3.3V, custom:Mini560-pro-3.3V, F.Cu at (219.4, 96.2)
- added U3: NRF24L01_Breakout, RF_Module:nRF24L01_Breakout, F.Cu at (152.1, 94.0)
- C1: footprint Capacitor_SMD:C_0201_0603Metric -> Capacitor_THT:CP_Radial_D8.0mm_P3.80mm
- moved C1 65.8 mm to (233.8, 80.2), turned to 180 degrees
- moved U1 18.9 mm to (150.3, 60.4)
- moved A1 7.33 mm to (191.0, 63.3)
- moved A2 5.51 mm to (222.0, 63.0)
- moved J6 5.05 mm to (178.3, 58.9)
- moved SW1 2.15 mm to (105.2, 63.5)
- moved SW2 2.15 mm to (105.2, 73.5)
- moved SW3 2.15 mm to (105.2, 84.0)
- moved SW4 1.58 mm to (105.0, 93.2)
- renumbered J3 to SW1, J2 to SW2, J1 to SW3, J4 to SW4, A3 to U1
Connections:
- net +12V renamed Net-(A1-VMOT)
- net GND1 renamed Net-(J7-Pin_2)
- A1 pad 14: Net-(A1-~{RESET}) -> Net-(A1-~{SLEEP})
- A2 pad 14: Net-(A2-~{RESET}) -> Net-(A2-~{SLEEP})
- U1 pad 17: Net-(A3-3V3) -> unconnected-(U1-3V3-Pad17)
Routing:
- net Net-(J7-Pin_2): track 199.2 -> 293.0 mm
- net Net-(U2-OUT-): track 0.00 -> 66.3 mm
- net Net-(A1-VMOT): track 104.2 -> 170.2 mm
- net Net-(U2-OUT+): track 0.00 -> 51.0 mm
- net Net-(A3-3V3): track 48.1 -> 0.00 mm
- net Net-(U1-D11): track 30.9 -> 68.8 mm
- net Net-(U1-D9): track 23.4 -> 58.3 mm
- net Net-(U1-D8): track 28.3 -> 53.5 mm
- net Net-(A2-~{SLEEP}): track 0.00 -> 18.4 mm
- net Net-(SW2-Pin_2): track 45.9 -> 27.6 mm
- net Net-(U1-D13): track 81.7 -> 63.6 mm, vias 2 -> 1
- net Net-(SW1-Pin_2): track 55.7 -> 38.6 mm
- net Net-(A2-STEP): track 80.6 -> 96.5 mm, vias 1 -> 0
- net Net-(U1-D12): track 48.1 -> 63.1 mm
- net Net-(A2-~{RESET}): track 0.00 -> 14.8 mm
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Other:
- board text added: "+"
- board text added: "12V"
- board text added: "3v3"
- board text added: "M1"
- board text added: "M2"

Commit message: Fixes
Parts:
- removed C6: 0.1mF, Capacitor_THT:C_Radial_D6.3mm_H7.0mm_P2.50mm
- removed C8: 100mF, Capacitor_THT:CP_Radial_D8.0mm_P3.80mm
- removed J6: Conn_01x04_Pin, Connector_PinHeader_2.54mm:PinHeader_1x04_P2.54mm_Vertical
- removed J8, J9, SW1, SW2, SW3, SW4: Conn_01x02_Pin, Connector_PinSocket_2.54mm:PinSocket_1x02_P2.54mm_Vertical
- removed U2: Mini560-pro-3.3V, custom:Mini560-pro-3.3V
- removed U3: NRF24L01_Breakout, RF_Module:nRF24L01_Breakout
- added C7: 10uF, Capacitor_THT:CP_Radial_D8.0mm_P3.80mm, F.Cu at (145.5, 82.1)
- added C9: 0.1uF, Capacitor_THT:C_Radial_D6.3mm_H7.0mm_P2.50mm, F.Cu at (145.6, 91.8)
- added J1: Conn_01x05_Pin, Connector_PinSocket_2.54mm:PinSocket_1x05_P2.54mm_Vertical, F.Cu at (116.8, 94.8)
- added J2: Conn_01x05_Pin, Connector_PinSocket_2.54mm:PinSocket_1x05_P2.54mm_Vertical, F.Cu at (103.4, 90.3)
- added J4: Conn_01x04_Pin, Connector_PinHeader_2.54mm:PinHeader_1x04_P2.54mm_Vertical, F.Cu at (211.5, 73.9)
- added SW5: Conn_01x02_Pin, Connector_PinSocket_2.54mm:PinSocket_1x02_P2.54mm_Vertical, F.Cu at (129.8, 88.3)
- added SW6: Conn_01x02_Pin, Connector_PinSocket_2.54mm:PinSocket_1x02_P2.54mm_Vertical, F.Cu at (119.8, 88.3)
- added SW7: Conn_01x02_Pin, Connector_PinSocket_2.54mm:PinSocket_1x02_P2.54mm_Vertical, F.Cu at (122.5, 93.3)
- added SW8: Conn_01x02_Pin, Connector_PinSocket_2.54mm:PinSocket_1x02_P2.54mm_Vertical, F.Cu at (131.1, 93.2)
- added U4: Mini560-pro-3.3V, custom:Mini560-pro-3.3V, F.Cu at (182.7, 94.9)
- added U5: NRF24L01_Breakout, RF_Module:nRF24L01_Breakout, F.Cu at (129.4, 69.3)
- C1: value 100mF -> 10uF
- C2: value 0.1mF -> 0.1uF
- C3: value 10mF -> 100mF
- C4: value 0.1mF -> 100mF; footprint Capacitor_THT:C_Radial_D6.3mm_H7.0mm_P2.50mm -> Capacitor_THT:CP_Radial_D8.0mm_P3.80mm
- C5: value 100mF -> 0.1uF; footprint Capacitor_THT:CP_Radial_D8.0mm_P3.80mm -> Capacitor_THT:C_Radial_D6.3mm_H7.0mm_P2.50mm; moved to B.Cu
- moved C5 62.3 mm to (134.4, 70.5), turned to -90 degrees
- moved C4 57.9 mm to (228.7, 90.9), turned to -90 degrees
- moved C3 46.7 mm to (223.2, 70.8)
- moved C1 38.9 mm to (196.0, 89.7)
- moved C2 38.0 mm to (186.3, 85.3)
- moved J5 37.3 mm to (215.8, 95.3), turned to -90 degrees
- moved A2 34.3 mm to (203.1, 91.6), turned to 90 degrees
- moved U1 32.8 mm to (183.0, 57.6)
- moved A1 10.2 mm to (198.7, 70.0), turned to 90 degrees
Connections:
- net Net-(A1-DIR) renamed /MOT1_DIR
- net Net-(A1-STEP) renamed /MOT1_STEP
- net Net-(A1-VDD) renamed +5V
- A1 pad 1: Net-(J7-Pin_2) -> GND
- A1 pad 14: Net-(A1-~{SLEEP}) -> Net-(A1-~{RESET})
- A1 pad 7: Net-(J7-Pin_2) -> GND
- A1 pad 8: Net-(A1-VMOT) -> +12V
- A2 pad 1: Net-(J7-Pin_2) -> GND
- A2 pad 14: Net-(A2-~{SLEEP}) -> Net-(A2-~{RESET})
- A2 pad 15: Net-(A2-STEP) -> /MOT2_STEP
- A2 pad 16: Net-(A2-DIR) -> /MOT2_DIR
- A2 pad 7: Net-(J7-Pin_2) -> GND
- A2 pad 8: Net-(A1-VMOT) -> +12V
- C1 pad 1: Net-(A1-VMOT) -> +12V
- C1 pad 2: Net-(J7-Pin_2) -> GND
- C2 pad 1: Net-(A1-VMOT) -> GND
- C2 pad 2: Net-(J7-Pin_2) -> +12V
- C3 pad 1: Net-(U2-OUT+) -> +12V
- C3 pad 2: Net-(U2-OUT-) -> GND
- C4 pad 1: Net-(U2-OUT+) -> +12V
- C4 pad 2: Net-(U2-OUT-) -> GND
- C5 pad 1: Net-(A1-VMOT) -> Net-(U4-OUT+)
- C5 pad 2: Net-(J7-Pin_2) -> Net-(U4-OUT-)
- J7 pad 1: Net-(A1-VMOT) -> +12V
- J7 pad 2: Net-(J7-Pin_2) -> GND
- U1 pad 1: unconnected-(U1-D1/TX-Pad1) -> /D1_TX
- U1 pad 11: Net-(U1-D8) -> /R_CE
- U1 pad 12: Net-(U1-D9) -> /R_CSN
- U1 pad 14: Net-(U1-D11) -> /R_MOSI
- U1 pad 15: Net-(U1-D12) -> /R_MISO
- U1 pad 16: Net-(U1-D13) -> /R_SCK
- U1 pad 17: unconnected-(U1-3V3-Pad17) -> +3.3V
- U1 pad 19: unconnected-(U1-A0-Pad19) -> /A0_Pin
- U1 pad 2: unconnected-(U1-D0/RX-Pad2) -> /D0_RX
- U1 pad 21: Net-(SW3-Pin_2) -> /LIM_S
- U1 pad 22: Net-(SW2-Pin_2) -> /LIM_N
- U1 pad 23: Net-(SW1-Pin_2) -> /LIM_E
- U1 pad 24: Net-(SW4-Pin_2) -> /LIM_W
- U1 pad 25: unconnected-(U1-A6-Pad25) -> /A6_Pin
- U1 pad 29: unconnected-(U1-GND-Pad29) -> GND
- U1 pad 30: Net-(A1-VMOT) -> +12V
- U1 pad 7: Net-(A2-STEP) -> /MOT2_DIR
- U1 pad 8: Net-(A2-DIR) -> /MOT2_STEP
- U1 pad 9: unconnected-(U1-D6-Pad9) -> /D6_Pin
Routing:
- net GND: track 0.00 -> 329.7 mm
- net Net-(J7-Pin_2): track 293.0 -> 0.00 mm
- net Net-(A1-VMOT): track 170.2 -> 0.00 mm
- net +12V: track 0.00 -> 142.7 mm
- net /D0_RX: track 0.00 -> 102.8 mm
- net /D1_TX: track 0.00 -> 101.9 mm, vias 0 -> 1
- net Net-(A2-DIR): track 101.2 -> 0.00 mm
- net Net-(A2-STEP): track 96.5 -> 0.00 mm
- net +5V: track 87.6 -> 171.7 mm, vias 1 -> 0
- net /D6_Pin: track 0.00 -> 73.7 mm, vias 0 -> 2
- net Net-(U4-OUT+): track 0.00 -> 71.7 mm
- net /A6_Pin: track 0.00 -> 69.3 mm, vias 0 -> 1
- net Net-(U1-D11): track 68.8 -> 0.00 mm
- net Net-(U2-OUT-): track 66.3 -> 0.00 mm
- net Net-(U1-D13): track 63.6 -> 0.00 mm, vias 1 -> 0
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Other:
- board text removed: "3v3"
- board text removed: "M1"
- board text removed: "M2"
