File: projects/Cat toy 1/wiring/box/limit_switches.kicad_sch (KiCad schematic)
At the start: 8 parts, among them SW5 Conn_01x02_Pin, SW6 Conn_01x02_Pin, SW7 Conn_01x02_Pin, SW8 Conn_01x02_Pin

Commit message: progress
Connections:
- no-connect marks 0 -> 4
