File: projects/Cat toy 1/wiring/box/motors.kicad_sch (KiCad schematic)
At the start: 8 parts, among them J4 Conn_01x04_Pin, J5 Conn_01x04_Pin, M1 Stepper_Motor_bipolar, M2 Stepper_Motor_bipolar

Commit message: progress
Connections:
- net +5V: now also A1.13 (~{RESET}), A1.14 (~{SLEEP}), A2.13 (~{RESET}), A2.14 (~{SLEEP})
- no-connect marks 0 -> 8
