File: projects/Cat toy 1/wiring/box/radio.kicad_sch (KiCad schematic)
At the start: 7 parts, among them U4 Mini560-pro-3.3V, U5 NRF24L01_Breakout

Commit message: progress
Connections:
- net GND: now also C5.2, C7.2, C9.2, U4.4 (OUT-), U5.1 (GND)
- net 3.3V: now reaches C5.1, C7.1, C9.1, U4.3 (OUT+), U5.2 (VCC)
