File: projects/Cat toy 1/wiring/box/wiring.kicad_pcb (KiCad board)
At the start: 2 copper layers, 136.9 x 42.3 mm, 21 parts, among them J1 Conn_01x05_Pin, J2 Conn_01x05_Pin, J4 Conn_01x04_Pin, J5 Conn_01x04_Pin, J7 Conn_01x02_Pin, SW5 Conn_01x02_Pin, SW6 Conn_01x02_Pin, SW7 Conn_01x02_Pin, SW8 Conn_01x02_Pin, U1 Arduino_Nano_v3.x, U4 Mini560-pro-3.3V, U5 NRF24L01_Breakout

Commit message: progress
Connections:
- net Net-(U4-OUT+) renamed /Radio/3.3V
- A1 pad 13: Net-(A1-~{RESET}) -> +5V
- A1 pad 14: Net-(A1-~{RESET}) -> +5V
- A2 pad 13: Net-(A2-~{RESET}) -> +5V
- A2 pad 14: Net-(A2-~{RESET}) -> +5V
- C5 pad 2: Net-(U4-OUT-) -> GND
- C7 pad 2: Net-(U4-OUT-) -> GND
- C9 pad 2: Net-(U4-OUT-) -> GND
- U4 pad 4: Net-(U4-OUT-) -> GND
- U5 pad 1: Net-(U4-OUT-) -> GND
Routing:
- net GND: track 329.7 -> 392.3 mm
- net Net-(U4-OUT-): track 59.3 -> 0.00 mm
- net +5V: track 171.7 -> 176.8 mm
- net Net-(A1-~{RESET}): track 2.54 -> 0.00 mm
- net Net-(A2-~{RESET}): track 2.54 -> 0.00 mm
