File: projects/Cat toy 1/wiring/box/wiring.kicad_sch (KiCad schematic)
At the start: 4 parts, among them J1 Conn_01x05_Pin, J2 Conn_01x05_Pin, J7 Conn_01x02_Pin, U1 Arduino_Nano_v3.x

Commit message: progress
Connections:
- net +12V: now also J7.1 (Pin_1), U1.30 (VIN)
- net 12V: no longer J7.1 (Pin_1), U1.30 (VIN)
- no-connect marks 0 -> 7
Other:
- moved on the sheet: J7
